File: hardware/bergara1.kicad_pcb (KiCad board)
At the start: 2 copper layers, 86.7 x 33.6 mm, 11 parts, among them J1 Screw_Terminal_01x02, SW1 SW_Nidec_CAS-120A1, U1 TA6586, U2 TA6586, U3 LM7805_TO220, U4 ESP32-C3_SUPERMINI_TH

Commit message: Hola
Connections:
- U4 pad 5: unconnected-(U4-GPIO5-Pad5) -> FI_2
- U4 pad 6: unconnected-(U4-GPIO6-Pad6) -> BI_2
- U4 pad 8: FI_2 -> unconnected-(U4-GPIO8-Pad8)
- U4 pad 9: BI_2 -> unconnected-(U4-GPIO9-Pad9)
Routing:
- net BI_2: track 8.25 -> 14.9 mm
- net FI_2: track 8.25 -> 14.6 mm
Changed lines of the file:
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@@
 	(net 18 "unconnected-(U4-GPIO0-Pad0)")
 	(net 19 "unconnected-(U4-GPIO2-Pad2)")
-	(net 20 "unconnected-(U4-GPIO5-Pad5)")
-	(net 21 "unconnected-(U4-GPIO6-Pad6)")
+	(net 20 "unconnected-(U4-GPIO8-Pad8)")
+	(net 21 "unconnected-(U4-GPIO9-Pad9)")
 	(net 22 "unconnected-(U4-GPIO21-Pad21)")
 	(net 23 "unconnected-(U4-GPIO20-Pad20)")
@@
 			(layers "*.Cu" "*.Mask")
 			(remove_unused_layers no)
-			(net 20 "unconnected-(U4-GPIO5-Pad5)")
+			(net 9 "FI_2")
 			(pinfunction "GPIO5")
 			(pintype "bidirectional")
@@
 			(layers "*.Cu" "*.Mask")
 			(remove_unused_layers no)
-			(net 21 "unconnected-(U4-GPIO6-Pad6)")
+			(net 10 "BI_2")
 			(pinfunction "GPIO6")
 			(pintype "bidirectional")
@@
 			(layers "*.Cu" "*.Mask")
 			(remove_unused_layers no)
-			(net 9 "FI_2")
+			(net 20 "unconnected-(U4-GPIO8-Pad8)")
 			(pinfunction "GPIO8")
 			(pintype "bidirectional")
@@
 			(layers "*.Cu" "*.Mask")
 			(remove_unused_layers no)
-			(net 10 "BI_2")
+			(net 21 "unconnected-(U4-GPIO9-Pad9)")
 			(pinfunction "GPIO9")
 			(pintype "bidirectional")
@@
 	)
 	(segment
+		(start 143.7036 55.0464)
+		(end 147.98 55.0464)
+		(width 1)
+		(layer "B.Cu")
+		(net 9)
+	)
+	(segment
 		(start 139.725 62.6664)
-		(end 147.98 62.6664)
+		(end 141.5836 62.6664)
+		(width 1)
+		(layer "B.Cu")
+		(net 9)
+	)
+	(segment
+		(start 142.5 56.25)
+		(end 143.7036 55.0464)
+		(width 1)
+		(layer "B.Cu")
+		(net 9)
+	)
+	(segment
+		(start 142.5 61.75)
+		(end 142.5 56.25)
+		(width 1)
+		(layer "B.Cu")
+		(net 9)
+	)
+	(segment
+		(start 141.5836 62.6664)
+		(end 142.5 61.75)
 		(width 1)
 		(layer "B.Cu")
@@
 	(segment
 		(start 139.725 65.2064)
-		(end 147.98 65.2064)
+		(end 143.5436 65.2064)
+		(width 1)
+		(layer "B.Cu")
+		(net 10)
+	)
+	(segment
+		(start 143.5436 65.2064)
+		(end 144.5 64.25)
+		(width 1)
+		(layer "B.Cu")
+		(net 10)
+	)
+	(segment
+		(start 145.1636 57.5864)
+		(end 147.98 57.5864)
+		(width 1)
+		(layer "B.Cu")
+		(net 10)
+	)
+	(segment
+		(start 144.5 64.25)
+		(end 144.5 58.25)
+		(width 1)
+		(layer "B.Cu")
+		(net 10)
+	)
+	(segment
+		(start 144.5 58.25)
+		(end 145.1636 57.5864)
 		(width 1)
 		(layer "B.Cu")
